File: CAD/PCB/Main/Main.kicad_pcb (KiCad board)
At the start: 2 copper layers, 65 x 56 mm, 9 parts, among them J1 GPIO, U2 MAX17320G20+T, U3 MCP3202T-CI/SN, U4 TPS56C230RJER, U5 VNH5019ATR-E

Commit message: Initial design
Parts:
- removed U2: MAX17320G20+T, RC_CAR:21-0139I_T2444-4_MXM-M
- removed U4: TPS56C230RJER, RC_CAR:RJE0020B
- added C14: 47uF, Resistor_SMD:R_1210_3225Metric_Pad1.30x2.65mm_HandSolder, F.Cu at (130.9, 66.0)
- added C2: 100nF, Resistor_SMD:R_0805_2012Metric_Pad1.20x1.40mm_HandSolder, F.Cu at (126.5, 51.5)
- added C20: 100nF, Resistor_SMD:R_0805_2012Metric_Pad1.20x1.40mm_HandSolder, F.Cu at (141.0, 53.0)
- added C23: 22uF, Resistor_SMD:R_1210_3225Metric_Pad1.30x2.65mm_HandSolder, F.Cu at (130.9, 69.5)
- added C24: 1uF, Resistor_SMD:R_1210_3225Metric_Pad1.30x2.65mm_HandSolder, F.Cu at (130.9, 62.5)
- added C25: 1uF, Resistor_SMD:R_1210_3225Metric_Pad1.30x2.65mm_HandSolder, F.Cu at (130.5, 79.0)
- added C26: 100nF, Resistor_SMD:R_0805_2012Metric_Pad1.20x1.40mm_HandSolder, F.Cu at (131.5, 72.5)
- added C27: 47uF, Resistor_SMD:R_1210_3225Metric_Pad1.30x2.65mm_HandSolder, F.Cu at (145.9, 74.5)
- added C28: 47uF, Resistor_SMD:R_1210_3225Metric_Pad1.30x2.65mm_HandSolder, F.Cu at (134.0, 79.0)
- added C29: 100nF, Resistor_SMD:R_0805_2012Metric_Pad1.20x1.40mm_HandSolder, F.Cu at (137.0, 78.5)
- added C3: 10uF, Resistor_SMD:R_0805_2012Metric_Pad1.20x1.40mm_HandSolder, F.Cu at (126.5, 53.5)
- added C30: 22uF, Resistor_SMD:R_1210_3225Metric_Pad1.30x2.65mm_HandSolder, F.Cu at (145.5, 78.0)
- added C31: 1uF, Resistor_SMD:R_1210_3225Metric_Pad1.30x2.65mm_HandSolder, F.Cu at (141.0, 78.5)
- added C32: 100nF, Resistor_SMD:R_0805_2012Metric_Pad1.20x1.40mm_HandSolder, F.Cu at (136.5, 75.5)
- added J2: XT60, Connector_AMASS:AMASS_XT60-M_1x02_P7.20mm_Vertical, F.Cu at (105.0, 67.5)
- added J3: XT30, Connector_AMASS:AMASS_XT30U-M_1x02_P5.0mm_Vertical, F.Cu at (123.0, 96.5)
- added J4: JST_PH, Connector_JST:JST_PH_B2B-PH-K_1x02_P2.00mm_Vertical, F.Cu at (139.0, 85.5)
- added J5: JST_PH, Connector_JST:JST_PH_B2B-PH-K_1x02_P2.00mm_Vertical, F.Cu at (139.0, 93.0)
- added J7: Conn_01x03, Connector_PinHeader_2.54mm:PinHeader_1x03_P2.54mm_Vertical, F.Cu at (135.5, 97.5)
- added Q1: IAUC100N04S6N015ATMA1, RC_CAR:IPC100N04S51R2ATMA1, F.Cu at (114.7, 55.4)
- added R10: 1k, Resistor_SMD:R_0805_2012Metric_Pad1.20x1.40mm_HandSolder, F.Cu at (124.5, 69.5)
- added R11: 1k, Resistor_SMD:R_0805_2012Metric_Pad1.20x1.40mm_HandSolder, F.Cu at (116.0, 68.0)
- added R12: 10k, Resistor_SMD:R_0805_2012Metric_Pad1.20x1.40mm_HandSolder, F.Cu at (121.0, 68.0)
- added R13: 1k, Resistor_SMD:R_0805_2012Metric_Pad1.20x1.40mm_HandSolder, F.Cu at (143.0, 53.0)
- added R14: 94k, Resistor_SMD:R_0805_2012Metric_Pad1.20x1.40mm_HandSolder, F.Cu at (106.0, 59.0)
- added R15: 1k, Resistor_SMD:R_0805_2012Metric_Pad1.20x1.40mm_HandSolder, F.Cu at (145.0, 53.0)
- added R16: 1k, Resistor_SMD:R_0805_2012Metric_Pad1.20x1.40mm_HandSolder, F.Cu at (147.0, 53.0)
- added R17: 10k, Resistor_SMD:R_0805_2012Metric_Pad1.20x1.40mm_HandSolder, F.Cu at (140.5, 73.5)
- added R18: 185, Resistor_SMD:R_0805_2012Metric_Pad1.20x1.40mm_HandSolder, F.Cu at (141.0, 59.5)
- added R19: 63.4k, Resistor_SMD:R_0805_2012Metric_Pad1.20x1.40mm_HandSolder, F.Cu at (144.0, 58.5)
- added R8: 1k, Resistor_SMD:R_0805_2012Metric_Pad1.20x1.40mm_HandSolder, F.Cu at (119.0, 68.0)
- added R9: 1k, Resistor_SMD:R_0805_2012Metric_Pad1.20x1.40mm_HandSolder, F.Cu at (123.5, 64.5)
- added S1: EG1271, RC_CAR:SW_EG1271, F.Cu at (105.0, 55.1)
- added TP3: MotorOutA, TestPoint:TestPoint_Pad_4.0x4.0mm, F.Cu at (129.5, 96.5)
- added TP4: MotorOutB, TestPoint:TestPoint_Pad_4.0x4.0mm, F.Cu at (111.5, 96.5)
- added U1: LMZ31707RVQR, RC_CAR:CONV_LMZ31707RVQR, F.Cu at (139.8, 66.4)
- moved U3 34.5 mm to (134.1, 53.9), turned to 180 degrees
- moved U5 19.9 mm to (119.5, 82.4), turned to -90 degrees
Connections:
- J1 pad 16: /GPIO23 -> Dir1
- J1 pad 18: /GPIO24 -> Dir2
- J1 pad 24: /GPIO8/SPI0.CE0 -> CS_0
- U3 pad 1: unconnected-(U3-*CS/SHDN-Pad1) -> CS_0
- U3 pad 2: unconnected-(U3-CH0-Pad2) -> ANALOG_IN_0
- U3 pad 3: unconnected-(U3-CH1-Pad3) -> ANALOG_IN_1
- U3 pad 4: unconnected-(U3-VSS-Pad4) -> GND
- U3 pad 5: unconnected-(U3-DIN-Pad5) -> /GPIO10/SPI0.MOSI
- U3 pad 6: unconnected-(U3-DOUT-Pad6) -> /GPIO9/SPI0.MISO
- U3 pad 7: unconnected-(U3-CLK-Pad7) -> /GPIO11/SPI0.SCLK
- U3 pad 8: unconnected-(U3-VDD/VREF-Pad8) -> +3V3
- U5 pad 1: unconnected-(U5-OUTA-Pad1) -> /MotorOutA
- U5 pad 10: unconnected-(U5-INB-Pad10) -> Net-(U5-INB)
- U5 pad 12: unconnected-(U5-VBAT-Pad12) -> VBATT
- U5 pad 13: unconnected-(U5-VCC-Pad13) -> VBATT
- U5 pad 15: unconnected-(U5-OUTB-Pad15) -> /MotorOutB
- U5 pad 16: unconnected-(U5-OUTB-Pad16) -> /MotorOutB
- U5 pad 18: unconnected-(U5-GNDB-Pad18) -> GND
- U5 pad 19: unconnected-(U5-GNDB-Pad19) -> GND
- U5 pad 20: unconnected-(U5-GNDB-Pad20) -> GND
- U5 pad 21: unconnected-(U5-OUTB-Pad21) -> /MotorOutB
- U5 pad 23: unconnected-(U5-VCC-Pad23) -> VBATT
- U5 pad 25: unconnected-(U5-OUTA-Pad25) -> /MotorOutA
- U5 pad 26: unconnected-(U5-GNDA-Pad26) -> GND
- U5 pad 27: unconnected-(U5-GNDA-Pad27) -> GND
- U5 pad 28: unconnected-(U5-GNDA-Pad28) -> GND
- U5 pad 3: unconnected-(U5-VCC-Pad3) -> VBATT
- U5 pad 30: unconnected-(U5-OUTA-Pad30) -> /MotorOutA
- U5 pad 31: unconnected-(U5-VCC-Pad31) -> VBATT
- U5 pad 32: unconnected-(U5-OUTA-Pad32) -> /MotorOutA
- U5 pad 33: unconnected-(U5-OUTB-Pad33) -> /MotorOutB
- U5 pad 4: unconnected-(U5-INA-Pad4) -> Net-(U5-INA)
- U5 pad 5: unconnected-(U5-ENA/DIAGA-Pad5) -> Net-(U5-ENA/DIAGA)
- U5 pad 6: unconnected-(U5-CS_DIS-Pad6) -> Net-(U5-CS_DIS)
- U5 pad 7: unconnected-(U5-PWM-Pad7) -> Net-(U5-PWM)
- U5 pad 8: unconnected-(U5-CS-Pad8) -> ANALOG_IN_0
- U5 pad 9: unconnected-(U5-ENB/DIAGB-Pad9) -> Net-(U5-ENA/DIAGA)
Routing:
- net VBATT: track 0.00 -> 125.0 mm
- net +5V: track 0.00 -> 120.7 mm, vias 0 -> 1
- net /GPIO13/PWM1: track 0.00 -> 112.1 mm
- net /MotorOutB: track 0.00 -> 64.2 mm, vias 0 -> 1
- net ANALOG_IN_0: track 0.00 -> 42.1 mm, vias 0 -> 2
- net /GPIO12/PWM0: track 0.00 -> 39.6 mm, vias 0 -> 1
- net /MotorOutA: track 0.00 -> 37.0 mm
- net Dir2: track 0.00 -> 28.6 mm, vias 0 -> 1
- net +3V3: track 0.00 -> 26.2 mm
- net Dir1: track 0.00 -> 23.8 mm
- net /AGND: track 0.00 -> 23.3 mm, vias 0 -> 2
- net Net-(J2-Pin_1): track 0.00 -> 21.5 mm
- net Net-(Q1-G): track 0.00 -> 19.4 mm
- net Net-(U5-ENA/DIAGA): track 0.00 -> 15.7 mm
- net GND: track 0.00 -> 15.1 mm
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- added copper zone on F.Cu, net unconnected-(U1-PH_10-Pad10)
Other:
- outline, holes or cut-outs redrawn
- copper layers 2 -> 4
- board text removed: "DISPLAY (OPTIONAL)"
- board text removed: "PoE"

Commit message: PCB almost done
Parts:
- removed MH4: MountingHole_2.7mm_M2.5, MountingHole:MountingHole_2.7mm_M2.5
- removed R15, R16: 1k, Resistor_SMD:R_0805_2012Metric_Pad1.20x1.40mm_HandSolder
- removed TP3: MotorOutA, TestPoint:TestPoint_Pad_4.0x4.0mm
- removed TP4: MotorOutB, TestPoint:TestPoint_Pad_4.0x4.0mm
- added 5V: GND, TestPoint:TestPoint_THTPad_D1.5mm_Drill0.7mm, F.Cu at (159.0, 67.3)
- added AIn: GND, TestPoint:TestPoint_THTPad_D1.5mm_Drill0.7mm, F.Cu at (162.8, 62.7)
- added C1: C_Polarized, Capacitor_SMD:CP_Elec_10x10, F.Cu at (137.9, 73.0)
- added C33: 1uF, Capacitor_SMD:C_0805_2012Metric_Pad1.18x1.45mm_HandSolder, F.Cu at (154.8, 61.3)
- added C34: 100nF, Capacitor_SMD:C_0805_2012Metric_Pad1.18x1.45mm_HandSolder, F.Cu at (153.2, 57.5)
- added C35: 1uF, Capacitor_SMD:C_0805_2012Metric_Pad1.18x1.45mm_HandSolder, F.Cu at (149.0, 51.5)
- added C36: 100nF, Capacitor_SMD:C_0805_2012Metric_Pad1.18x1.45mm_HandSolder, F.Cu at (149.2, 57.5)
- added C4: C_Polarized, Capacitor_SMD:CP_Elec_10x10, F.Cu at (137.9, 84.0)
- added C5: C_Polarized, Capacitor_SMD:CP_Elec_6.3x7.7, F.Cu at (105.0, 85.0)
- added CS_1: GND, TestPoint:TestPoint_THTPad_D1.5mm_Drill0.7mm, F.Cu at (162.8, 54.0)
- added GND: GND, TestPoint:TestPoint_THTPad_D1.5mm_Drill0.7mm, F.Cu at (135.8, 98.2)
- added GND: GND, TestPoint:TestPoint_THTPad_D1.5mm_Drill0.7mm, F.Cu at (159.0, 62.7)
- added GND: GND, TestPoint:TestPoint_THTPad_D1.5mm_Drill0.7mm, F.Cu at (162.8, 67.2)
- added J6: JST_PH, Connector_JST:JST_PH_B2B-PH-K_1x02_P2.00mm_Vertical, F.Cu at (139.5, 93.1)
- added MISO: GND, TestPoint:TestPoint_THTPad_D1.5mm_Drill0.7mm, F.Cu at (162.8, 58.0)
- added MOSI: GND, TestPoint:TestPoint_THTPad_D1.5mm_Drill0.7mm, F.Cu at (158.9, 58.0)
- added MotorA: MotorOutA, TestPoint:TestPoint_Pad_4.0x4.0mm, F.Cu at (130.0, 96.0)
- added MotorB: MotorOutB, TestPoint:TestPoint_Pad_4.0x4.0mm, F.Cu at (111.0, 96.0)
- added SCL: GND, TestPoint:TestPoint_THTPad_D1.5mm_Drill0.7mm, F.Cu at (158.8, 54.0)
- added VBatt: GND, TestPoint:TestPoint_THTPad_D1.5mm_Drill0.7mm, F.Cu at (140.8, 98.4)
- C14, C23, C27, C28, C30: footprint Resistor_SMD:R_1210_3225Metric_Pad1.30x2.65mm_HandSolder -> Capacitor_SMD:C_1210_3225Metric_Pad1.33x2.70mm_HandSolder
- C2, C20, C26, C29, C32: footprint Resistor_SMD:R_0805_2012Metric_Pad1.20x1.40mm_HandSolder -> Capacitor_SMD:C_0805_2012Metric_Pad1.18x1.45mm_HandSolder
- C24, C25, C31: footprint Resistor_SMD:R_1210_3225Metric_Pad1.30x2.65mm_HandSolder -> Capacitor_SMD:C_0805_2012Metric_Pad1.18x1.45mm_HandSolder
- C3: value 10uF -> 1uF; footprint Resistor_SMD:R_0805_2012Metric_Pad1.20x1.40mm_HandSolder -> Capacitor_SMD:C_0805_2012Metric_Pad1.18x1.45mm_HandSolder
- R13: value 1k -> 1.5k
- moved J7 46.3 mm to (152.8, 54.5), turned to -90 degrees
- moved J5 32.9 mm to (150.8, 62.2), turned to 180 degrees
- moved C28 31.7 mm to (104.4, 90.5), turned to 180 degrees
- moved R8 27.3 mm to (145.0, 59.8)
- moved J4 20.6 mm to (150.8, 68.5), turned to 180 degrees
- moved C14 18.9 mm to (117.1, 53.2)
- moved C23 18.9 mm to (117.1, 56.7)
- moved R18 18.0 mm to (124.2, 53.1), turned to 0 degrees
- moved C26 17.9 mm to (117.1, 61.8)
- moved C29 16.3 mm to (133.0, 62.7), turned to -90 degrees
- moved R19 16.1 mm to (128.8, 53.1), turned to 180 degrees
- moved U1 15.1 mm to (125.9, 60.5)
- moved C30 15.1 mm to (139.2, 64.3)
- moved R17 14.7 mm to (126.8, 68.2), turned to -90 degrees
- moved C24 14.2 mm to (117.1, 59.6)
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Connections:
- net /AGND renamed AGND
- net /GPIO10/SPI0.MOSI renamed MOSI
- net /GPIO11/SPI0.SCLK renamed SCL
- net /GPIO12/PWM0 renamed PWM_0
- net /GPIO13/PWM1 renamed PWM_1
- net /GPIO9/SPI0.MISO renamed MISO
- net /MotorOutA renamed MotorOutA
- net /MotorOutB renamed MotorOutB
- net ANALOG_IN_0 renamed Analog_In_0
- net VBATT renamed VBatt
- J1 pad 16: Dir1 -> Dir_2
- J1 pad 18: Dir2 -> Dir_1
- J1 pad 26: /GPIO7/SPI0.CE1 -> CS_1
- R10 pad 2: Dir1 -> Dir_1
- R11 pad 1: Dir2 -> Dir_2
- R13 pad 1: Net-(R13-Pad1) -> GND
- U3 pad 3: ANALOG_IN_1 -> Analog_In_1
Routing:
- net PWM_1: track 112.1 -> 7.92 mm
- net +3V3: track 26.2 -> 85.5 mm, vias 0 -> 2
- net +5V: track 120.7 -> 158.1 mm, vias 1 -> 11
- net MOSI: track 3.41 -> 37.1 mm
- net MISO: track 6.39 -> 40.1 mm
- net Dir_2: track 0.00 -> 29.2 mm, vias 0 -> 1
- net Analog_In_1: track 0.00 -> 28.6 mm, vias 0 -> 1
- net Dir2: track 28.6 -> 0.00 mm, vias 1 -> 0
- net CS_1: track 0.00 -> 28.3 mm
- net PWM_0: track 39.6 -> 13.1 mm
- net MotorOutA: track 37.0 -> 62.8 mm, vias 0 -> 2
- net Dir_1: track 0.00 -> 25.3 mm, vias 0 -> 1
- net SCL: track 8.71 -> 33.0 mm
- net Dir1: track 23.8 -> 0.00 mm
- net Net-(U5-PWM): track 4.93 -> 28.5 mm, vias 0 -> 2
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- added copper zone on F.Cu, net +5V
- added copper zone on B.Cu, net GND
- added copper zone on F.Cu, net GND
- added copper zone on In1.Cu, net GND
- added copper zone on In2.Cu, net GND
- added copper zone on F.Cu, net Net-(J2-Pin_1)
- added copper zone on In1.Cu, net Net-(J2-Pin_1)
- added copper zone on F.Cu, net VBatt
Other:
- outline, holes or cut-outs redrawn
- board text added: "MC-LTX 2026"
- board text removed: "CAMERA (OPTIONAL)"
- board text removed: "Extend PCB edge 0.5mm if using SMT header"
- board text removed: "RJ45"
- board text removed: "USB"

Commit message: pcb order is in
Parts:
- removed J2: XT60, Connector_AMASS:AMASS_XT60-M_1x02_P7.20mm_Vertical
- removed Q1: IAUC100N04S6N015ATMA1, RC_CAR:IPC100N04S51R2ATMA1
- removed R14: 94k, Resistor_SMD:R_0805_2012Metric_Pad1.20x1.40mm_HandSolder
- removed S1: EG1271, RC_CAR:SW_EG1271
- added D1: D_Zener_Filled, Diode_SMD:D_SOD-123F, F.Cu at (144.4, 53.8)
- added IC1: BTS70021EPPXUMA1, RC_CAR:SOP65P600X115-15N, F.Cu at (107.1, 78.1)
- added J8: XT60, Connector_AMASS:AMASS_XT60-M_1x02_P7.20mm_Vertical, F.Cu at (105.7, 63.0)
- added JP1: SolderJumper_2_Open, Jumper:SolderJumper-2_P1.3mm_Open_RoundedPad1.0x1.5mm, F.Cu at (156.3, 51.5)
- added R20: 4.7k, Resistor_SMD:R_0805_2012Metric_Pad1.20x1.40mm_HandSolder, F.Cu at (101.5, 79.0)
- added R21: 94k, Resistor_SMD:R_0805_2012Metric_Pad1.20x1.40mm_HandSolder, F.Cu at (138.8, 63.1)
- added R22: 35k, Resistor_SMD:R_0805_2012Metric_Pad1.20x1.40mm_HandSolder, F.Cu at (138.8, 61.0)
- added R23: 10k, Resistor_SMD:R_0805_2012Metric_Pad1.20x1.40mm_HandSolder, F.Cu at (111.5, 53.1)
- added S2: EG1271, RC_CAR:SW_EG1271, F.Cu at (105.8, 54.3)
- moved C30 1.50 mm to (139.3, 65.8)
- moved U3 1.13 mm to (136.8, 53.6)
- moved C20 1.06 mm to (142.2, 55.2)
- moved C27 0.70 mm to (144.2, 65.0)
- moved C32 0.30 mm to (135.3, 62.7)
- moved C35 0.20 mm to (149.0, 51.7)
- moved R8 0.20 mm to (145.2, 59.8)
- renumbered 5V to +5V, GND to 3V3, AIn to GND
Connections:
- GND pad 1: Analog_In_1 -> GND
Routing:
- net Net-(IC1-VS): track 0.00 -> 47.4 mm, vias 0 -> 4
- net GND: track 21.7 -> 64.6 mm, vias 44 -> 50
- net Net-(IC1-IN): track 0.00 -> 32.4 mm, vias 0 -> 2
- net Net-(JP1-A): track 0.00 -> 26.9 mm, vias 0 -> 2
- net VBatt: track 140.1 -> 157.4 mm, vias 3 -> 8
- net Net-(Q1-G): track 15.3 -> 0.00 mm
- net Net-(R23-Pad1): track 0.00 -> 12.2 mm
- net Analog_In_1: track 28.6 -> 19.7 mm, vias 1 -> 0
- net Analog_In_0: track 36.8 -> 41.4 mm
- net Net-(IC1-DEN): track 0.00 -> 3.13 mm
- net MOSI: track 37.1 -> 36.0 mm
- net MISO: track 40.1 -> 39.4 mm
- added copper zone on F.Cu, net Net-(IC1-VS)
- removed copper zone on F.Cu, net Net-(J2-Pin_1)
- removed copper zone on In1.Cu, net Net-(J2-Pin_1)
Other:
- board text added: "PWM"
- board text added: "V0"
