File: CAD/PCB/Main/Main.kicad_sch (KiCad schematic)
At the start: 10 parts, among them J1 GPIO, U1 CAT24C256, U2 MAX17320G20+T, U3 MCP3202T-CI/SN, U4 TPS56C230RJER, U5 VNH5019ATR-E

Commit message: Initial design
Parts:
- removed C1: 100n, symbol Device:C_Small
- removed JP1: ID_WP, symbol Jumper:SolderJumper_2_Open
- removed R1, R2: 3.9k, symbol Device:R_Small
- removed U1: CAT24C256, symbol Memory_EEPROM:CAT24C256
- removed U2: MAX17320G20+T, RC_CAR:21-0139I_T2444-4_MXM-M, symbol RC_CAR:MAX17320G20+T
- added C10, C16, C19, C2, C20, C26, C29, C32, C4: 100nF, Resistor_SMD:R_0805_2012Metric_Pad1.20x1.40mm_HandSolder, symbol Device:C
- added C11, C12, C13, C18, C23, C30: 22uF, Resistor_SMD:R_1210_3225Metric_Pad1.30x2.65mm_HandSolder, symbol Device:C
- added C14, C27, C28, C6, C7, C8, C9: 47uF, Resistor_SMD:R_1210_3225Metric_Pad1.30x2.65mm_HandSolder, symbol Device:C
- added C15, C17, C24, C25, C31, C5: 1uF, Resistor_SMD:R_1210_3225Metric_Pad1.30x2.65mm_HandSolder, symbol Device:C
- added C21, C22: 22pF, Resistor_SMD:R_0805_2012Metric_Pad1.20x1.40mm_HandSolder, symbol Device:C
- added C3: 10uF, Resistor_SMD:R_0805_2012Metric_Pad1.20x1.40mm_HandSolder, symbol Device:C
- added J2: XT60, Connector_AMASS:AMASS_XT60-M_1x02_P7.20mm_Vertical, symbol Connector_Generic:Conn_01x02
- added J3: XT30, Connector_AMASS:AMASS_XT30U-M_1x02_P5.0mm_Vertical, symbol Connector_Generic:Conn_01x02
- added J4, J5: JST_PH, Connector_JST:JST_PH_B2B-PH-K_1x02_P2.00mm_Vertical, symbol Connector_Generic:Conn_01x02
- added J7: Conn_01x03, Connector_PinHeader_2.54mm:PinHeader_1x03_P2.54mm_Vertical, symbol Connector_Generic:Conn_01x03
- added L1: 1.8uH, Inductor_SMD:L_Wuerth_HCI-1050, symbol Device:L
- added Q1: IAUC100N04S6N015ATMA1, RC_CAR:IPC100N04S51R2ATMA1, symbol RC_CAR:IAUC100N04S6N015ATMA1
- added R10, R11, R13, R15, R16, R8, R9: 1k, Resistor_SMD:R_0805_2012Metric_Pad1.20x1.40mm_HandSolder, symbol Device:R
- added R12, R17: 10k, Resistor_SMD:R_0805_2012Metric_Pad1.20x1.40mm_HandSolder, symbol Device:R
- added R14, R3, R5: 94k, Resistor_SMD:R_0805_2012Metric_Pad1.20x1.40mm_HandSolder, symbol Device:R
- added R18: 185, Resistor_SMD:R_0805_2012Metric_Pad1.20x1.40mm_HandSolder, symbol Device:R
- added R19: 63.4k, Resistor_SMD:R_0805_2012Metric_Pad1.20x1.40mm_HandSolder, symbol Device:R
- added R4: 12k, Resistor_SMD:R_0805_2012Metric_Pad1.20x1.40mm_HandSolder, symbol Device:R
- added R6: 180k, Resistor_SMD:R_0805_2012Metric_Pad1.20x1.40mm_HandSolder, symbol Device:R
- added R7: 33k, Resistor_SMD:R_0805_2012Metric_Pad1.20x1.40mm_HandSolder, symbol Device:R
- added S1: EG1271, RC_CAR:SW_EG1271, symbol RC_CAR:EG1271
- added TP1, TP5, TP6: GND, TestPoint:TestPoint_Pad_3.0x3.0mm, symbol Connector:TestPoint
- added TP10: AnalogIn1, TestPoint:TestPoint_Pad_3.0x3.0mm, symbol Connector:TestPoint
- added TP12: VBATT, TestPoint:TestPoint_Pad_3.0x3.0mm, symbol Connector:TestPoint
- added TP13: MOSI, TestPoint:TestPoint_Pad_3.0x3.0mm, symbol Connector:TestPoint
- added TP14: MISO, TestPoint:TestPoint_Pad_3.0x3.0mm, symbol Connector:TestPoint
- added TP15: SCL, TestPoint:TestPoint_Pad_3.0x3.0mm, symbol Connector:TestPoint
- added TP16: CS_1, TestPoint:TestPoint_Pad_3.0x3.0mm, symbol Connector:TestPoint
- added TP2: +3V3, TestPoint:TestPoint_Pad_3.0x3.0mm, symbol Connector:TestPoint
- added TP3: MotorOutA, TestPoint:TestPoint_Pad_4.0x4.0mm, symbol Connector:TestPoint
- added TP4: MotorOutB, TestPoint:TestPoint_Pad_4.0x4.0mm, symbol Connector:TestPoint
- added TP7, TP8, TP9: +5V, TestPoint:TestPoint_Pad_3.0x3.0mm, symbol Connector:TestPoint
- added U1: LMZ31707RVQR, RC_CAR:CONV_LMZ31707RVQR, symbol RC_CAR:LMZ31707RVQR
Connections:
- net GPIO8/SPI0.CE0 is gone; now on net CS_0: J1.24 (Pin_24)
- net +3V3: now also U3.8 (VDD/VREF), C2.1, C3.1, R9.2, TP2.1
- net +5V: now also C13.2, C14.1, C15.2, C16.2, C21.2, C22.2, C23.1, C24.1, C26.1, C6.2, C7.2, C8.2, C9.2, J4.1 (Pin_1), J5.1 (Pin_1), J7.2 (Pin_2), L1.2, R17.2, R3.1, TP7.1, TP8.1, TP9.1, U1.27 (SENSE+), U1.34 (VOUT_34), U1.35 (VOUT_35), U1.36 (VOUT_36), U1.37 (VOUT_37), U1.38 (VOUT_38), U1.41 (VOUT_41)
- net GND: now also U3.4 (VSS), U4.10 (NC), U4.13 (AGND), U4.16 (NC), U4.18 (PGND), U4.21 (PGND), U4.7 (PGND), U4.8 (PGND), U5.14 (NC), U5.17 (NC), U5.18 (GNDB), U5.19 (GNDB), U5.2 (NC), U5.20 (GNDB), U5.22 (NC), U5.24 (NC), U5.26 (GNDA), U5.27 (GNDA), U5.28 (GNDA), U5.29 (NC), C10.2, C11.2, C12.2, C13.1, C14.2, C15.1, C16.1, C17.2, C18.2, C19.2, C2.2, C20.1, C23.2, C24.2, C25.1, C26.2, C27.2, C28.2, C29.1, C3.2, C30.2, C31.2, C32.2, C5.2, C6.1, C7.1, C8.1, C9.1, J4.2 (Pin_2), J5.2 (Pin_2), J7.3 (Pin_3), Q1.5 (D_1), Q1.6 (D_2), Q1.7 (D_3), Q1.8 (D_4), Q1.9 (D_5), R12.2, R15.1, R16.1, R4.2, R7.1, TP1.1, TP5.1, TP6.1, U1.20 (PGND_20), U1.21 (PGND_21), U1.31 (PGND_31), U1.32 (PGND_32), U1.33 (PGND_33)
- net GPIO10/SPI0.MOSI: now also U3.5 (DIN), TP13.1
- net GPIO11/SPI0.SCLK: now also U3.7 (CLK), TP15.1
- net GPIO12/PWM0: now also R8.2
- net GPIO13/PWM1: now also J7.1 (Pin_1)
- net GPIO7/SPI0.CE1: now also TP16.1
- net GPIO9/SPI0.MISO: now also U3.6 (DOUT), TP14.1
- net at U4.1 (BST): now also C4.2
- net VCC: now reaches U4.12 (EN)
- net VCC: now also U4.17 (VCC), C19.1, C5.1, R5.2, R6.1
- net at U4.14 (FB): now also C21.1, C22.1, R3.2, R4.1
- net at U4.15 (MODE): now also R6.2, R7.2
- net at U4.19 (SW): now also U4.20 (SW), U4.6 (SW), C4.1, L1.1
- net VBATT: now reaches U4.2 (VIN)
- net VBATT: now also U4.3 (VIN), U4.4 (VIN), U4.5 (VIN), U5.12 (VBAT), U5.13 (VCC), U5.23 (VCC), U5.3 (VCC), U5.31 (VCC), C10.1, C11.1, C12.1, C17.1, C18.1, C25.2, C27.1, C28.1, C29.2, C30.1, C31.1, C32.1, J2.2 (Pin_2), S1.1, S1.4, TP12.1, U1.1 (PVIN_1), U1.11 (PVIN_11), U1.12 (PVIN_12), U1.3 (VIN), U1.39 (PVIN_39), U1.40 (PVIN_40)
- net at U4.9 (PGOOD): now also R5.1
- net MotorOutA: now reaches U5.1 (OUTA)
- net MotorOutA: now also U5.25 (OUTA), U5.30 (OUTA), U5.32 (OUTA), J3.1 (Pin_1), TP3.1
- net at U5.10 (INB): now also R11.2
- net MotorOutB: now reaches U5.15 (OUTB)
- net MotorOutB: now also U5.16 (OUTB), U5.21 (OUTB), U5.33 (OUTB), J3.2 (Pin_2), TP4.1
- net at U5.4 (INA): now also R10.1
- net at U5.5 (ENA/DIAGA): now also U5.9 (ENB/DIAGB), R9.1
- net at U5.6 (CS_DIS): now also R12.1
- net at U5.7 (PWM): now also R8.1
- net ANALOG_IN_0: now reaches U5.8 (CS)
- net ANALOG_IN_0: now also U3.2 (CH0), C20.2, R13.2
- net CS_0: now reaches U3.1 (*CS/SHDN)
- net ANALOG_IN_1: now reaches U3.3 (CH1)
- net ANALOG_IN_1: now also TP10.1
- net GPIO23 renamed Dir1
- net Dir1: now also R10.2
- net GPIO24 renamed Dir2
- net Dir2: now also R11.1
- new net: R13.1, R15.2, R16.2
- new net: Q1.4 (G), R14.1, S1.2, S1.5
- new net: J2.1 (Pin_1), Q1.1 (S_1), Q1.10 (S_4), Q1.2 (S_2), Q1.3 (S_3), R14.2
- new net: R18.2, U1.26 (VADJ)
- new net: U1.10 (PH_10), U1.13 (PH_13), U1.14 (PH_14), U1.15 (PH_15), U1.16 (PH_16), U1.17 (PH_17), U1.18 (PH_18), U1.19 (PH_19), U1.42 (PH_42), U1.43 (PH_42__1), U1.44 (PH_42__2), U1.45 (PH_42__3), U1.46 (PH_42__4), U1.47 (PH_42__5), U1.48 (PH_42__6), U1.49 (PH_42__7), U1.50 (PH_42__8), U1.51 (PH_42__9), U1.52 (PH_42__10), U1.53 (PH_42__11), U1.54 (PH_42__12), U1.55 (PH_42__13), U1.56 (PH_42__14)
- new net: R19.1, U1.22 (RT/CLK)
- new net: R17.1, U1.8 (PWRGD)
- new net AGND: R18.1, R19.2, U1.2 (AGND_2), U1.23 (AGND_23), U1.29 (STSEL)
- no-connect marks 3 -> 34
Other:
- note removed: "Additional pin functions: https://pinout.xyz/"
- note removed: "ID_SD and ID_SC PINS: These pins are reserved for HAT ID EEPROM. At boot time this I2C interface will be interrogated to look for an EEPROM that identifes the attached board and allows automagic setup of the GPIOs (and optionally, Linux drivers). Bridging JP1 enables write protection. DO NOT USE these pins for anything other than attaching an I2C ID EEPROM. Leave unconnected if ID EEPROM not requ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"
- title: (none) -> RC_CAR
- moved on the sheet: U3, U4, U5

Commit message: PCB almost done
Parts:
- removed C10, C16, C19, C4: 100nF, Resistor_SMD:R_0805_2012Metric_Pad1.20x1.40mm_HandSolder, symbol Device:C
- removed C11, C12, C13, C18: 22uF, Resistor_SMD:R_1210_3225Metric_Pad1.30x2.65mm_HandSolder, symbol Device:C
- removed C15, C17, C5: 1uF, Resistor_SMD:R_1210_3225Metric_Pad1.30x2.65mm_HandSolder, symbol Device:C
- removed C21, C22: 22pF, Resistor_SMD:R_0805_2012Metric_Pad1.20x1.40mm_HandSolder, symbol Device:C
- removed C6, C7, C8, C9: 47uF, Resistor_SMD:R_1210_3225Metric_Pad1.30x2.65mm_HandSolder, symbol Device:C
- removed L1: 1.8uH, Inductor_SMD:L_Wuerth_HCI-1050, symbol Device:L
- removed R15, R16: 1k, Resistor_SMD:R_0805_2012Metric_Pad1.20x1.40mm_HandSolder, symbol Device:R
- removed R3, R5: 94k, Resistor_SMD:R_0805_2012Metric_Pad1.20x1.40mm_HandSolder, symbol Device:R
- removed R4: 12k, Resistor_SMD:R_0805_2012Metric_Pad1.20x1.40mm_HandSolder, symbol Device:R
- removed R6: 180k, Resistor_SMD:R_0805_2012Metric_Pad1.20x1.40mm_HandSolder, symbol Device:R
- removed R7: 33k, Resistor_SMD:R_0805_2012Metric_Pad1.20x1.40mm_HandSolder, symbol Device:R
- removed TP1, TP5, TP6: GND, TestPoint:TestPoint_Pad_3.0x3.0mm, symbol Connector:TestPoint
- removed TP10: AnalogIn1, TestPoint:TestPoint_Pad_3.0x3.0mm, symbol Connector:TestPoint
- removed TP13: MOSI, TestPoint:TestPoint_Pad_3.0x3.0mm, symbol Connector:TestPoint
- removed TP14: MISO, TestPoint:TestPoint_Pad_3.0x3.0mm, symbol Connector:TestPoint
- removed TP15: SCL, TestPoint:TestPoint_Pad_3.0x3.0mm, symbol Connector:TestPoint
- removed TP16: CS_1, TestPoint:TestPoint_Pad_3.0x3.0mm, symbol Connector:TestPoint
- removed TP2: +3V3, TestPoint:TestPoint_Pad_3.0x3.0mm, symbol Connector:TestPoint
- removed TP7, TP8, TP9: +5V, TestPoint:TestPoint_Pad_3.0x3.0mm, symbol Connector:TestPoint
- removed U4: TPS56C230RJER, RC_CAR:RJE0020B, symbol RC_CAR:TPS56C230RJER
- added 5V1, CS_1, GND1, GND2, GND3, MISO1, MOSI1, SCL1, VBatt1: GND, TestPoint:TestPoint_THTPad_D1.5mm_Drill0.7mm, symbol Connector:TestPoint
- added C1, C4: C_Polarized, Capacitor_SMD:CP_Elec_10x10, symbol Device:C_Polarized
- added C33, C35: 1uF, Capacitor_SMD:C_0805_2012Metric_Pad1.18x1.45mm_HandSolder, symbol Device:C
- added C34, C36: 100nF, Capacitor_SMD:C_0805_2012Metric_Pad1.18x1.45mm_HandSolder, symbol Device:C
- added C5: C_Polarized, Capacitor_SMD:CP_Elec_6.3x7.7, symbol Device:C_Polarized
- added J6: JST_PH, Connector_JST:JST_PH_B2B-PH-K_1x02_P2.00mm_Vertical, symbol Connector_Generic:Conn_01x02
- C14, C23, C27, C28, C30: footprint Resistor_SMD:R_1210_3225Metric_Pad1.30x2.65mm_HandSolder -> Capacitor_SMD:C_1210_3225Metric_Pad1.33x2.70mm_HandSolder
- C2, C20, C26, C29, C32: footprint Resistor_SMD:R_0805_2012Metric_Pad1.20x1.40mm_HandSolder -> Capacitor_SMD:C_0805_2012Metric_Pad1.18x1.45mm_HandSolder
- C24, C25, C31: footprint Resistor_SMD:R_1210_3225Metric_Pad1.30x2.65mm_HandSolder -> Capacitor_SMD:C_0805_2012Metric_Pad1.18x1.45mm_HandSolder
- C3: value 10uF -> 1uF; footprint Resistor_SMD:R_0805_2012Metric_Pad1.20x1.40mm_HandSolder -> Capacitor_SMD:C_0805_2012Metric_Pad1.18x1.45mm_HandSolder
- R13: value 1k -> 1.5k
- TP12: value VBATT -> GND; footprint TestPoint:TestPoint_Pad_3.0x3.0mm -> TestPoint:TestPoint_THTPad_D1.5mm_Drill0.7mm
- renumbered TP3 to MotorA1, TP4 to MotorB1
Connections:
- net +3V3: now also GND3.1
- net +5V: now also 5V1.1, C33.2, C34.2, C35.2, C36.2
- net GND: now also R13.1, C1.2, C33.1, C34.1, C35.1, C36.1, C4.2, C5.2, GND1.1, GND2.1, J6.2 (Pin_2); no longer U5.14 (NC), U5.17 (NC), U5.2 (NC), U5.29 (NC)
- net ANALOG_IN_0 renamed Analog_In_0
- net ANALOG_IN_1 renamed Analog_In_1
- net Analog_In_1: now also TP12.1
- net Dir1 renamed Dir_1
- net Dir_1: now also J1.18 (Pin_18); no longer J1.16 (Pin_16)
- net Dir2 renamed Dir_2
- net Dir_2: now also J1.16 (Pin_16); no longer J1.18 (Pin_18)
- net GPIO10/SPI0.MOSI renamed MOSI
- net MOSI: now also MOSI1.1
- net GPIO11/SPI0.SCLK renamed SCL
- net SCL: now also SCL1.1
- net GPIO12/PWM0 renamed PWM_0
- net GPIO13/PWM1 renamed PWM_1
- net GPIO7/SPI0.CE1 renamed CS_1
- net CS_1: now also CS_1.1
- net GPIO9/SPI0.MISO renamed MISO
- net MISO: now also MISO1.1
- net VBATT renamed VBatt
- net VBatt: now also C1.1, C4.1, C5.1, J6.1 (Pin_1), VBatt1.1; no longer TP12.1
- no-connect marks 34 -> 37
Other:
- moved on the sheet: C14, C20, C23, C24, C25, C26, C27, C28, C29, C30, C31, C32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

Commit message: pcb order is in
Parts:
- removed J2: XT60, Connector_AMASS:AMASS_XT60-M_1x02_P7.20mm_Vertical, symbol Connector_Generic:Conn_01x02
- removed Q1: IAUC100N04S6N015ATMA1, RC_CAR:IPC100N04S51R2ATMA1, symbol RC_CAR:IAUC100N04S6N015ATMA1
- removed R14: 94k, Resistor_SMD:R_0805_2012Metric_Pad1.20x1.40mm_HandSolder, symbol Device:R
- removed S1: EG1271, RC_CAR:SW_EG1271, symbol RC_CAR:EG1271
- added D1: D_Zener_Filled, Diode_SMD:D_SOD-123F, symbol Device:D_Zener_Filled
- added IC1: BTS70021EPPXUMA1, RC_CAR:SOP65P600X115-15N, symbol RC_CAR:BTS70021EPPXUMA1
- added J8: XT60, Connector_AMASS:AMASS_XT60-M_1x02_P7.20mm_Vertical, symbol Connector_Generic:Conn_01x02
- added JP1: SolderJumper_2_Open, Jumper:SolderJumper-2_P1.3mm_Open_RoundedPad1.0x1.5mm, symbol Jumper:SolderJumper_2_Open
- added R20: 4.7k, Resistor_SMD:R_0805_2012Metric_Pad1.20x1.40mm_HandSolder, symbol Device:R
- added R21: 180k, Resistor_SMD:R_0805_2012Metric_Pad1.20x1.40mm_HandSolder, symbol Device:R
- added R22: 63.4k, Resistor_SMD:R_0805_2012Metric_Pad1.20x1.40mm_HandSolder, symbol Device:R
- added R23: 10k, Resistor_SMD:R_0805_2012Metric_Pad1.20x1.40mm_HandSolder, symbol Device:R
- added S2: EG1271, RC_CAR:SW_EG1271, symbol RC_CAR:EG1271
- R18: value 185 -> 187
Connections:
- net Analog_In_0: now also D1.1 (K)
- net Analog_In_1: now also JP1.2 (B); no longer TP12.1
- net GND: now also TP12.1, D1.2 (A), IC1.1 (GND), J8.1 (Pin_1), R20.2, R22.1
- net VBatt: now also IC1.10 (OUT_3), IC1.12 (OUT_4), IC1.13 (OUT_5), IC1.14 (OUT_6), IC1.8 (OUT_1), IC1.9 (OUT_2), R21.2
- new net: R23.1, S2.1, S2.4
- new net: IC1.2 (IN), R23.2
- new net: JP1.1 (A), R21.1, R22.2
- new net: IC1.15 (VS), J8.2 (Pin_2), S2.2, S2.5
- new net: IC1.3 (DEN), R20.1
- no-connect marks 37 -> 42
Other:
- moved on the sheet: 5V1, C1, C14, C2, C20, C23, C24, C25, C26, C27, C28, C29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
